Commit message: set effort and velocity to non-zero

File: assets/x500/x500.urdf (robot description, URDF)
Before this commit: robot x500-Base, 5 links, 4 joints
Joints:
- joint x500-Base__rotor_0_joint: limit lower=-1e+16 upper=1e+16 effort=0.0 velocity=0.0 -> lower=-1e+16 upper=1e+16 effort=1.0 velocity=1.0
- joint x500-Base__rotor_1_joint: limit lower=-1e+16 upper=1e+16 effort=0.0 velocity=0.0 -> lower=-1e+16 upper=1e+16 effort=1.0 velocity=1.0
- joint x500-Base__rotor_2_joint: limit lower=-1e+16 upper=1e+16 effort=0.0 velocity=0.0 -> lower=-1e+16 upper=1e+16 effort=1.0 velocity=1.0
- joint x500-Base__rotor_3_joint: limit lower=-1e+16 upper=1e+16 effort=0.0 velocity=0.0 -> lower=-1e+16 upper=1e+16 effort=1.0 velocity=1.0
